File: eagle/tinyha_meas.sch (EAGLE design)
At the start: 38 parts, among them IC1 MCP16301, IC2 ATMEGA88PA-AU, IC3 ST485ECDR, Q1 FDV301N, Q2 FDV301N, Q3 FDV301N, Q7 FDV301N, X1 ILCX13-FF5F18-16.0000

Commit message: SVN revision 1367
Other:
- note added: "TCRT5000L LED-A LED-C T-C T-E"
Changed lines of the file:
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@@
 <?xml version="1.0" encoding="utf-8"?>
 <!DOCTYPE eagle SYSTEM "eagle.dtd">
-<eagle version="7.7.0">
+<eagle version="7.5.0">
 <drawing>
 <settings>
@@
 <sheet>
 <plain>
-<text x="249.174" y="156.972" size="1.4224" layer="96">SFH229 C</text>
-<text x="249.174" y="154.432" size="1.4224" layer="96">SFH229 A</text>
-<text x="249.174" y="151.892" size="1.4224" layer="96">LED A</text>
-<text x="249.174" y="149.352" size="1.4224" layer="96">LED C</text>
+<text x="249.174" y="151.892" size="1.4224" layer="96">SFH229 C</text>
+<text x="249.174" y="149.352" size="1.4224" layer="96">SFH229 A</text>
+<text x="249.174" y="156.972" size="1.4224" layer="96">LED A</text>
+<text x="249.174" y="154.432" size="1.4224" layer="96">LED C</text>
+<text x="261.62" y="149.86" size="1.6764" layer="96">TCRT5000L
+LED-A
+LED-C
+T-C
+T-E</text>
 </plain>
 <instances>
@@
 </schematic>
 </drawing>
+<compatibility>
+<note version="6.3" minversion="6.2.2" severity="warning">
+Since Version 6.2.2 text objects can contain more than one line,
+which will not be processed correctly with this version.
+</note>
+</compatibility>
 </eagle>
